Commit message: add testdrone mesh

File: tools/Simulation/src/bmflight_simulation/urdf/bmflight_test_drone.xacro (robot description, xacro)
@@ -6,12 +6,13 @@
   <xacro:property name="rotor_velocity_slowdown_sim" value="10" />
   <xacro:property name="use_mesh_file" value="true" />
-  <xacro:property name="mesh_file" value="package://bmflight_simulation/meshes/heisl.dae" />
+  <xacro:property name="mesh_file" value="package://bmflight_simulation/meshes/bmflight_test_drone.dae" />
   <xacro:property name="mass" value="0.68" /> <!-- [kg] -->
-  <xacro:property name="body_width" value="0.1" /> <!-- [m] -->
-  <xacro:property name="body_height" value="0.12" /> <!-- [m] -->
+  <xacro:property name="body_width" value="0.08" /> <!-- [m] -->
+  <xacro:property name="body_height" value="0.06" /> <!-- [m] -->
   <xacro:property name="mass_rotor" value="0.009" /> <!-- [kg] -->
-  <xacro:property name="arm_length" value="0.17" /> <!-- [m] -->
-  <xacro:property name="rotor_offset_top" value="0.01" /> <!-- [m] -->
-  <xacro:property name="radius_rotor" value="0.1" /> <!-- [m] -->
+  <xacro:property name="rotor_offset_top" value="0.018" /> <!-- [m] -->
+  <xacro:property name="arm_length_x" value="0.0848" /> <!-- [m] -->
+  <xacro:property name="arm_length_y" value="0.1015" /> <!-- [m] -->
+  <xacro:property name="radius_rotor" value="0.06" /> <!-- [m] -->
   <xacro:property name="motor_constant" value="8.54858e-06" /> <!-- [kg m/s^2] -->
   <xacro:property name="moment_constant" value="0.016" /> <!-- [m] -->
@@ -44,6 +45,6 @@
   <xacro:vertical_rotor
     robot_namespace="${namespace}"
-    suffix="front"
-    direction="cw"
+    suffix="front_right"
+    direction="ccw"
     motor_constant="${motor_constant}"
     moment_constant="${moment_constant}"
@@ -60,11 +61,11 @@
     use_own_mesh="false"
     mesh="">
-    <origin xyz="${arm_length} 0 ${rotor_offset_top}" rpy="0 0 0" />
+    <origin xyz="${arm_length_x} -${arm_length_y} ${rotor_offset_top}" rpy="0 0 0" />
     <xacro:insert_block name="rotor_inertia" />
   </xacro:vertical_rotor>
   <xacro:vertical_rotor
     robot_namespace="${namespace}"
-    suffix="left"
-    direction="ccw"
+    suffix="front_left"
+    direction="cw"
     motor_constant="${motor_constant}"
     moment_constant="${moment_constant}"
@@ -78,14 +79,14 @@
     rotor_drag_coefficient="${rotor_drag_coefficient}"
     rolling_moment_coefficient="${rolling_moment_coefficient}"
-    color="Blue"
+    color="Red"
     use_own_mesh="false"
     mesh="">
-    <origin xyz="0 ${arm_length} ${rotor_offset_top}" rpy="0 0 0" />
+    <origin xyz="${arm_length_x} ${arm_length_y} ${rotor_offset_top}" rpy="0 0 0" />
     <xacro:insert_block name="rotor_inertia" />
   </xacro:vertical_rotor>
   <xacro:vertical_rotor
     robot_namespace="${namespace}"
-    suffix="back"
-    direction="cw"
+    suffix="back_left"
+    direction="ccw"
     motor_constant="${motor_constant}"
     moment_constant="${moment_constant}"
@@ -102,11 +103,11 @@
     use_own_mesh="false"
     mesh="">
-    <origin xyz="-${arm_length} 0 ${rotor_offset_top}" rpy="0 0 0" />
+    <origin xyz="-${arm_length_x} ${arm_length_y} ${rotor_offset_top}" rpy="0 0 0" />
     <xacro:insert_block name="rotor_inertia" />
   </xacro:vertical_rotor>
   <xacro:vertical_rotor
     robot_namespace="${namespace}"
-    suffix="right"
-    direction="ccw"
+    suffix="back_right"
+    direction="cw"
     motor_constant="${motor_constant}"
     moment_constant="${moment_constant}"
@@ -123,5 +124,5 @@
     use_own_mesh="false"
     mesh="">
-    <origin xyz="0 -${arm_length} ${rotor_offset_top}" rpy="0 0 0" />
+    <origin xyz="-${arm_length_x} -${arm_length_y} ${rotor_offset_top}" rpy="0 0 0" />
     <xacro:insert_block name="rotor_inertia" />
   </xacro:vertical_rotor>

Commit message: adapt mixer to yaw inverse

File: tools/Simulation/src/bmflight_simulation/urdf/bmflight_test_drone.xacro (robot description, xacro)
@@ -7,5 +7,5 @@
   <xacro:property name="use_mesh_file" value="true" />
   <xacro:property name="mesh_file" value="package://bmflight_simulation/meshes/bmflight_test_drone.dae" />
-  <xacro:property name="mass" value="0.68" /> <!-- [kg] -->
+  <xacro:property name="mass" value="0.88" /> <!-- [kg] -->
   <xacro:property name="body_width" value="0.08" /> <!-- [m] -->
   <xacro:property name="body_height" value="0.06" /> <!-- [m] -->

Commit message: update simulation

File: tools/Simulation/src/bmflight_simulation/urdf/bmflight_test_drone.xacro (robot description, xacro)
@@ -1,6 +1,4 @@
 <?xml version="1.0"?>
 <robot name="bmflight_test_drone" xmlns:xacro="http://ros.org/wiki/xacro">
-  <!-- Properties (Taken from Novel Dynamic Inversion Architecture Design
-for Quadrocopter Control by Jian Wang et al.) -->
   <xacro:property name="namespace" value="$(arg namespace)" />
   <xacro:property name="rotor_velocity_slowdown_sim" value="10" />
@@ -10,5 +8,5 @@
   <xacro:property name="body_width" value="0.08" /> <!-- [m] -->
   <xacro:property name="body_height" value="0.06" /> <!-- [m] -->
-  <xacro:property name="mass_rotor" value="0.009" /> <!-- [kg] -->
+  <xacro:property name="mass_rotor" value="0.005" /> <!-- [kg] -->
   <xacro:property name="rotor_offset_top" value="0.018" /> <!-- [m] -->
   <xacro:property name="arm_length_x" value="0.0848" /> <!-- [m] -->
@@ -24,9 +22,9 @@
   <!-- Property Blocks -->
   <xacro:property name="body_inertia">
-    <inertia ixx="0.007" ixy="0.0" ixz="0.0" iyy="0.007" iyz="0.0" izz="0.012" /> <!-- [kg m^2] [kg m^2] [kg m^2] [kg m^2] [kg m^2] [kg m^2] -->
+    <inertia ixx="0.002815882266667" ixy="0.0" ixz="0.0" iyy="0.001085115477333" iyz="0.0" izz="0.003813904410667" /> <!-- [kg m^2] [kg m^2] [kg m^2] [kg m^2] [kg m^2] [kg m^2] -->
   </xacro:property>
-  <!-- inertia of a single rotor, assuming it is a cuboid. Height=3mm, width=15mm -->
+  <!-- inertia of a single rotor, assuming it is a cuboid. Height=5m, width=15mm -->
   <xacro:property name="rotor_inertia">
-    <xacro:box_inertia x="${radius_rotor}" y="0.015" z="0.003" mass="${mass_rotor*rotor_velocity_slowdown_sim}" />
+    <xacro:box_inertia x="${radius_rotor}" y="0.015" z="0.005" mass="${mass_rotor*rotor_velocity_slowdown_sim}" />
   </xacro:property>
   <!-- Included URDF Files -->
