Commit message: add odementry

File: tools/Simulation/src/bmflight_simulation/urdf/bmflightTest.xacro (robot description, xacro)
@@ -6,27 +6,52 @@
     <!-- Instantiate a controller. -->
     <xacro:controller_plugin_macro namespace="${namespace}" imu_sub_topic="imu" />
-    <xacro:if value="$(arg enable_mavlink_interface)">
-        <!-- Instantiate mavlink telemetry interface. -->
-        <xacro:default_mavlink_interface namespace="${namespace}" imu_sub_topic="imu" rotor_count="4" />
-    </xacro:if>
-    <!-- Mount an ADIS16448 IMU. -->
+    <!-- Mount an ideal IMU. -->
     <xacro:imu_plugin_macro
         namespace="${namespace}"
-        imu_suffix=""
-        parent_link="${namespace}/base_link"
-        imu_topic="imu"
-        mass_imu_sensor="0.015"
-        measurement_divisor="1"
-        measurement_delay="0"
-        gyroscope_noise_density="0.0"
-        gyroscope_random_walk="0.0"
-        gyroscope_bias_correlation_time="1000.0"
-        gyroscope_turn_on_bias_sigma="0.000"
-        accelerometer_noise_density="0.001180"
-        accelerometer_random_walk="0.000"
-        accelerometer_bias_correlation_time="300.0"
-        accelerometer_turn_on_bias_sigma="0.0">
+	    imu_suffix=""
+	    parent_link="${namespace}/base_link"
+	    imu_topic="imu"
+	    measurement_delay="0"
+	    measurement_divisor="1"
+	    mass_imu_sensor="0.00001"
+	    gyroscope_noise_density="0.0"
+	    gyroscope_random_walk="0.0"
+	    gyroscope_bias_correlation_time="1000.0"
+	    gyroscope_turn_on_bias_sigma= "0.0"
+	    accelerometer_noise_density="0.0"
+	    accelerometer_random_walk="0.0"
+	    accelerometer_bias_correlation_time="300.0"
+	    accelerometer_turn_on_bias_sigma="0">
         <inertia ixx="0.00001" ixy="0.0" ixz="0.0" iyy="0.00001" iyz="0.0" izz="0.00001" />
         <origin xyz="0 0 0" rpy="0 0 0" />
     </xacro:imu_plugin_macro>
+	<xacro:odometry_plugin_macro
+	    namespace="${namespace}"
+	    odometry_sensor_suffix="1"
+	    parent_link="${namespace}/base_link"
+	    pose_topic="odometry_sensor1/pose"
+	    pose_with_covariance_topic="odometry_sensor1/pose_with_covariance"
+	    position_topic="odometry_sensor1/position"
+	    transform_topic="odometry_sensor1/transform"
+	    odometry_topic="odometry_sensor1/odometry"
+	    parent_frame_id="world"
+	    child_frame_id="${namespace}/odometry_sensor1"
+	    mass_odometry_sensor="0.00001"
+	    measurement_divisor="1"
+	    measurement_delay="0"
+	    unknown_delay="0.0"
+	    noise_normal_position="0 0 0"
+	    noise_normal_quaternion="0 0 0"
+	    noise_normal_linear_velocity="0 0 0"
+	    noise_normal_angular_velocity="0 0 0"
+	    noise_uniform_position="0 0 0"
+	    noise_uniform_quaternion="0 0 0"
+	    noise_uniform_linear_velocity="0 0 0"
+	    noise_uniform_angular_velocity="0 0 0"
+	    enable_odometry_map="false"
+	    odometry_map=""
+	    image_scale="">
+	    <inertia ixx="0.00001" ixy="0.0" ixz="0.0" iyy="0.00001" iyz="0.0" izz="0.00001" /> <!-- [kg m^2] [kg m^2] [kg m^2] [kg m^2] [kg m^2] [kg m^2] -->
+	    <origin xyz="0.0 0.0 0.0" rpy="0.0 0.0 0.0" />
+  	</xacro:odometry_plugin_macro>
 </robot>

File: tools/Simulation/src/bmflight_simulation/urdf/bmflight_test_drone.xacro (robot description, xacro)
@@ -6,5 +6,5 @@
   <xacro:property name="rotor_velocity_slowdown_sim" value="10" />
   <xacro:property name="use_mesh_file" value="true" />
-  <xacro:property name="mesh_file" value="package://bmflight_simulation/meshes/bmflight_test_drone.dae" />
+  <xacro:property name="mesh_file" value="package://bmflight_simulation/meshes/heisl.dae" />
   <xacro:property name="mass" value="0.68" /> <!-- [kg] -->
   <xacro:property name="body_width" value="0.1" /> <!-- [m] -->

Commit message: fix interia and add macro for tof and fpv camera

File: tools/Simulation/src/bmflight_simulation/urdf/bmflightTest.xacro (robot description, xacro)
@@ -55,3 +55,138 @@
 	    <origin xyz="0.0 0.0 0.0" rpy="0.0 0.0 0.0" />
   	</xacro:odometry_plugin_macro>
+	<!-- Macro to add a tof sensor. -->
+    <xacro:macro name="tof_plugin_macro"
+        params="namespace tof_suffix parent_link tof_topic mass_tof_sensor *inertia *origin">
+        <!-- tof link -->
+        <link name="${namespace}/tof${tof_suffix}_link">
+            <inertial>
+                <xacro:insert_block name="inertia" />
+                <mass value="${mass_tof_sensor}" />  <!-- [kg] -->
+                <origin xyz="0 0 0" rpy="0 0 0" />
+            </inertial>
+            <visual>
+                <geometry>
+                    <box size="0.004 0.02 0.015"/>
+                </geometry>
+            </visual>
+        </link>
+        <!-- tof joint -->
+        <joint name="${namespace}/tof${tof_suffix}_joint" type="revolute">
+            <xacro:insert_block name="origin" />
+            <parent link="${parent_link}" />
+            <child link="${namespace}/tof${tof_suffix}_link" />
+            <limit upper="0" lower="0" effort="0" velocity="0" />
+        </joint>
+        <gazebo reference="${namespace}/tof${tof_suffix}_link">
+            <material>Gazebo/Red</material>
+            <sensor name="laser" type="ray">
+                <pose>0 0 0 0 0 0</pose>
+                <ray>
+                    <scan>
+                    <horizontal>
+                        <samples>1</samples>
+                        <resolution>1</resolution>
+                        <min_angle>-0</min_angle>
+                        <max_angle>0</max_angle>
+                    </horizontal>
+                    </scan>
+                    <range>
+                        <min>0.002</min>
+                        <max>2</max>
+                        <resolution>0.001</resolution>
+                    </range>
+                    <noise>
+                        <type>gaussian</type>
+                        <mean>0.0</mean>
+                        <stddev>0.001</stddev>
+                    </noise>
+                </ray>
+                <plugin name="${namespace}/tof${tof_suffix}_plugin" filename="libgazebo_ros_laser.so">
+                    <robotNamespace>${namespace}</robotNamespace>
+                    <topicName>${tof_topic}</topicName>
+                    <frameName>${namespace}/tof${tof_suffix}_link</frameName>
+                </plugin>
+                <always_on>1</always_on>
+                <update_rate>33</update_rate>
+                <visualize>true</visualize>
+            </sensor>
+        </gazebo>
+    </xacro:macro>
+    <!--<xacro:tof_plugin_macro
+        namespace="${namespace}"
+        tof_suffix="_ground"
+        parent_link="${namespace}/base_link"
+        tof_topic="tof_ground_sensor"
+        mass_tof_sensor="0.00001">
+        <inertia ixx="0.00000" ixy="0.0" ixz="0.0" iyy="0.00000" iyz="0.0" izz="0.00000" />
+        <origin xyz="0.00 0 0" rpy="0 0 0" />
+    </xacro:tof_plugin_macro>
+    -->
+  	<!-- Macro to add a camera rgb camera. -->
+    <xacro:macro name="camera_macro"
+        params="namespace camera_suffix parent_link camera_topic mass_camera_sensor *inertia *origin">
+        <!-- camera link -->
+        <link name="${namespace}/camera${camera_suffix}_link">
+            <inertial>
+                <xacro:insert_block name="inertia" />
+                <mass value="${mass_camera_sensor}" />  <!-- [kg] -->
+                <origin xyz="0 0 0" rpy="0 0 0" />
+            </inertial>
+            <visual>
+                <geometry>
+                    <box size="0.004 0.02 0.015"/>
+                </geometry>
+            </visual>
+        </link>
+        <!-- camera joint -->
+        <joint name="${namespace}/camera${camera_suffix}_joint" type="revolute">
+            <xacro:insert_block name="origin" />
+            <parent link="${parent_link}" />
+            <child link="${namespace}/camera${camera_suffix}_link" />
+            <limit upper="0" lower="0" effort="0" velocity="0" />
+        </joint>
+        <gazebo reference="${namespace}/camera${camera_suffix}_link">
+            <material>Gazebo/Red</material>
+            <sensor name='camera1' type='camera'>
+			    <camera name="head">
+			      <horizontal_fov>1.3962634</horizontal_fov>
+			      <image>
+			        <width>800</width>
+			        <height>800</height>
+			        <format>R8G8B8</format>
+			      </image>
+			      <clip>
+			        <near>0.02</near>
+			        <far>300</far>
+			      </clip>
+			    </camera>
+			    <always_on>1</always_on>
+			    <update_rate>30</update_rate>
+			    <visualize>1</visualize>
+			    <plugin name="{namespace}/camera${camera_suffix}_plugin" filename="libgazebo_ros_camera.so">
+				    <alwaysOn>true</alwaysOn>
+				    <updateRate>0.0</updateRate>
+				    <cameraName>${camera_topic}/camera</cameraName>
+				    <imageTopicName>${camera_topic}/image_raw</imageTopicName>
+				    <cameraInfoTopicName>${camera_topic}/camera_info</cameraInfoTopicName>
+				    <frameName>${namespace}/camera${camera_suffix}_link</frameName>
+				    <hackBaseline>0.07</hackBaseline>
+				    <distortionK1>0.0</distortionK1>
+				    <distortionK2>0.0</distortionK2>
+				    <distortionK3>0.0</distortionK3>
+				    <distortionT1>0.0</distortionT1>
+				    <distortionT2>0.0</distortionT2>
+			  	</plugin>
+			</sensor>
+        </gazebo>
+    </xacro:macro>
+  	<!--<xacro:camera_macro
+        namespace="${namespace}"
+        camera_suffix="_front"
+        parent_link="${namespace}/base_link"
+        camera_topic="fpv"
+        mass_camera_sensor="0.00001">
+        <inertia ixx="0.00001" ixy="0.0" ixz="0.0" iyy="0.00001" iyz="0.0" izz="0.00001" />
+        <origin xyz="0.1 0 0.01" rpy="0 0 0" />
+    </xacro:camera_macro>-->
 </robot>

File: tools/Simulation/src/bmflight_simulation/urdf/bmflight_test_drone.xacro (robot description, xacro)
@@ -7,5 +7,5 @@
   <xacro:property name="mass" value="0.88" /> <!-- [kg] -->
   <xacro:property name="body_width" value="0.08" /> <!-- [m] -->
-  <xacro:property name="body_height" value="0.06" /> <!-- [m] -->
+  <xacro:property name="body_height" value="0.04" /> <!-- [m] -->
   <xacro:property name="mass_rotor" value="0.005" /> <!-- [kg] -->
   <xacro:property name="rotor_offset_top" value="0.018" /> <!-- [m] -->
@@ -22,5 +22,6 @@
   <!-- Property Blocks -->
   <xacro:property name="body_inertia">
-    <inertia ixx="0.002815882266667" ixy="0.0" ixz="0.0" iyy="0.001085115477333" iyz="0.0" izz="0.003813904410667" /> <!-- [kg m^2] [kg m^2] [kg m^2] [kg m^2] [kg m^2] [kg m^2] -->
+   <!-- [kg m^2] [kg m^2] [kg m^2] [kg m^2] [kg m^2] [kg m^2] -->
+    <inertia ixx="0.001438548933333" ixy="0.0" ixz="0.0" iyy="0.002462448810667" iyz="0.0" izz="0.003813904410667" />
   </xacro:property>
   <!-- inertia of a single rotor, assuming it is a cuboid. Height=5m, width=15mm -->

Commit message: mount sensors

File: tools/Simulation/src/bmflight_simulation/urdf/bmflightTest.xacro (robot description, xacro)
@@ -113,5 +113,5 @@
         </gazebo>
     </xacro:macro>
-    <!--<xacro:tof_plugin_macro
+    <xacro:tof_plugin_macro
         namespace="${namespace}"
         tof_suffix="_ground"
@@ -119,8 +119,43 @@
         tof_topic="tof_ground_sensor"
         mass_tof_sensor="0.00001">
-        <inertia ixx="0.00000" ixy="0.0" ixz="0.0" iyy="0.00000" iyz="0.0" izz="0.00000" />
-        <origin xyz="0.00 0 0" rpy="0 0 0" />
-    </xacro:tof_plugin_macro>
-    -->
+        <inertia ixx="0.00001" ixy="0.0" ixz="0.0" iyy="0.00001" iyz="0.0" izz="0.00001" />
+        <origin xyz="0.10 0 0" rpy="0 ${pi/2} 0" />
+    </xacro:tof_plugin_macro>
+ <!--    <xacro:tof_plugin_macro
+        namespace="${namespace}"
+        tof_suffix="_front"
+        parent_link="${namespace}/base_link"
+        tof_topic="tof_front_sensor"
+        mass_tof_sensor="0.20">
+        <inertia ixx="0.00001" ixy="0.0" ixz="0.0" iyy="0.00001" iyz="0.0" izz="0.00001" />
+        <origin xyz="0.12 0 0" rpy="0 0 0" />
+    </xacro:tof_plugin_macro>
+   <xacro:tof_plugin_macro
+        namespace="${namespace}"
+        tof_suffix="_right"
+        parent_link="${namespace}/base_link"
+        tof_topic="tof_right_sensor"
+        mass_tof_sensor="0.00001">
+        <inertia ixx="0.00001" ixy="0.0" ixz="0.0" iyy="0.00001" iyz="0.0" izz="0.00001" />
+        <origin xyz="0 0.045 0" rpy="0 0 ${pi/2}" />
+    </xacro:tof_plugin_macro>
+	<xacro:tof_plugin_macro
+        namespace="${namespace}"
+        tof_suffix="_left"
+        parent_link="${namespace}/base_link"
+        tof_topic="tof_left_sensor"
+        mass_tof_sensor="0.00001">
+        <inertia ixx="0.00001" ixy="0.0" ixz="0.0" iyy="0.00001" iyz="0.0" izz="0.00001" />
+        <origin xyz="0 -0.045 0" rpy="0 0 -${pi/2}" />
+    </xacro:tof_plugin_macro>
+    <xacro:tof_plugin_macro
+        namespace="${namespace}"
+        tof_suffix="_back"
+        parent_link="${namespace}/base_link"
+        tof_topic="tof_back_sensor"
+        mass_tof_sensor="0.00001">
+        <inertia ixx="0.00001" ixy="0.0" ixz="0.0" iyy="0.00001" iyz="0.0" izz="0.00001" />
+        <origin xyz="-0.1 0 0" rpy="0 0 -${pi}" />
+    </xacro:tof_plugin_macro>-->
   	<!-- Macro to add a camera rgb camera. -->
     <xacro:macro name="camera_macro"
